File: CH340E-10P.sch (KiCad schematic (older format))
At the start: 7 parts, among them U4 CH340E

Commit message: test push
Parts:
- gave numbers to parts that had none: 3
Other:
- note added: "Best for 5V Communication"
- note removed: "Best for 3.3V Communication"
Changed lines of the file:
@@
 P 4400 2650
 AR Path="/601CCEA4/6023C445" Ref="D?"  Part="1"
-AR Path="/601CD882/6023C445" Ref="D?"  Part="1"
-F 0 "D?" V 4300 2500 50  0000 C CNN
+AR Path="/601CD882/6023C445" Ref="D2"  Part="1"
+F 0 "D2" V 4300 2500 50  0000 C CNN
 F 1 "1N5819WS" V 4400 2375 50  0000 C CNN
 F 2 "Diode_SMD:D_SOD-323" V 4400 2650 50  0001 C CNN
@@
 P 4400 3100
 AR Path="/601CCEA4/6023C44E" Ref="F?"  Part="1"
-AR Path="/601CD882/6023C44E" Ref="F?"  Part="1"
-F 0 "F?" H 4350 3000 50  0000 L CNN
+AR Path="/601CD882/6023C44E" Ref="F2"  Part="1"
+F 0 "F2" H 4350 3000 50  0000 L CNN
 F 1 "500mA" H 4275 3175 50  0000 L CNN
 F 2 "Fuse:Fuse_1206_3216Metric" H 4400 3100 50  0001 C CNN
@@
 P 4350 3850
 AR Path="/601CCEA4/6023C454" Ref="#PWR?"  Part="1"
-AR Path="/601CD882/6023C454" Ref="#PWR?"  Part="1"
-F 0 "#PWR?" H 4350 3600 50  0001 C CNN
+AR Path="/601CD882/6023C454" Ref="#PWR0103"  Part="1"
+F 0 "#PWR0103" H 4350 3600 50  0001 C CNN
 F 1 "GND" H 4355 3677 50  0000 C CNN
 F 2 "" H 4350 3850 50  0001 C CNN
@@
 	4400 2400 4400 2550
 $Comp
-L Power_Protection:USBLC6-2SC6 U?
+L Power_Protection:USBLC6-2SC6 U3
 U 1 1 6023C460
 P 5400 3650
-AR Path="/601CD882/6023C460" Ref="U?"  Part="1"
+AR Path="/601CD882/6023C460" Ref="U3"  Part="1"
 AR Path="/601CCEA4/6023C460" Ref="U?"  Part="1"
-F 0 "U?" V 5750 3450 50  0000 C CNN
+F 0 "U3" V 5750 3450 50  0000 C CNN
 F 1 "USBLC6-2SC6" V 5050 3200 50  0000 C CNN
 F 2 "Package_TO_SOT_SMD:SOT-23-6" H 5400 3150 50  0001 C CNN
@@
 P 5850 3650
 AR Path="/601CCEA4/6023C46A" Ref="#PWR?"  Part="1"
-AR Path="/601CD882/6023C46A" Ref="#PWR?"  Part="1"
-F 0 "#PWR?" H 5850 3400 50  0001 C CNN
+AR Path="/601CD882/6023C46A" Ref="#PWR0107"  Part="1"
+F 0 "#PWR0107" H 5850 3400 50  0001 C CNN
 F 1 "GND" V 5855 3522 50  0000 R CNN
 F 2 "" H 5850 3650 50  0001 C CNN
@@
 D-
 Text Notes 4050 4450 0    50   ~ 0
-Best for 3.3V Communication
+Best for 5V Communication
 $Comp
-L power:PWR_FLAG #FLG?
+L power:PWR_FLAG #FLG0102
 U 1 1 6025701C
 P 4850 2750
-F 0 "#FLG?" H 4850 2825 50  0001 C CNN
+F 0 "#FLG0102" H 4850 2825 50  0001 C CNN
 F 1 "PWR_FLAG" H 4850 2923 50  0000 C CNN
 F 2 "" H 4850 2750 50  0001 C CNN
